File: CUT_OFF/CUT_OFF_MODULE.kicad_sch (KiCad schematic)
At the start: 52 parts, among them IC1 4011N, IC2 4538N, J1 CONNECTOR, Q1 BC307, Q2 BD140, T1 BC547, T2 BC547, T3 BC337

Commit message: KiCad project of cut-off module updated
Changed lines of the file:
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@@
 (kicad_sch
-	(version 20231120)
+	(version 20250114)
 	(generator "eeschema")
-	(generator_version "8.0")
+	(generator_version "9.0")
 	(paper "A3")
 	(title_block
 		(title "CUT-OFF MODULE")
 		(date "04.06.2018")
+		(rev "A")
 		(company "trwgQ26xxx")
 	)
+	(text "THROTTLE CLOSED CONFIRM?"
+		(exclude_from_sim no)
+		(at 370.84 85.09 0)
+		(effects
+			(font
+				(size 1.778 1.5113)
+			)
+			(justify left bottom)
+		)
+	)
+	(text "IC1 = 4011"
+		(exclude_from_sim no)
+		(at 119.888 72.39 0)
+		(effects
+			(font
+				(size 1.5113 1.5113)
+			)
+		)
+	)
+	(text "IC2 = 4538"
+		(exclude_from_sim no)
+		(at 177.292 82.55 0)
+		(effects
+			(font
+				(size 1.5113 1.5113)
+			)
+		)
+	)
 	(junction
 		(at 299.72 133.35)
@@
 		)
 	)
-	(text "THROTTLE CLOSED CONFIRM?"
-		(exclude_from_sim no)
-		(at 370.84 85.09 0)
-		(effects
-			(font
-				(size 1.778 1.5113)
-			)
-			(justify left bottom)
-		)
-	)
-	(text "IC1 = 4011"
-		(exclude_from_sim no)
-		(at 119.888 72.39 0)
-		(effects
-			(font
-				(size 1.5113 1.5113)
-			)
-		)
-	)
-	(text "IC2 = 4538"
-		(exclude_from_sim no)
-		(at 177.292 82.55 0)
-		(effects
-			(font
-				(size 1.5113 1.5113)
-			)
-		)
-	)
 	(global_label "P3_GROUND"
 		(shape input)
@@
 		)
 	)
+	(embedded_fonts no)
 )
