File: ESD_48/ESD_48.kicad_sch (KiCad schematic)
At the start: 14 parts, among them J1 PWR, U1 HEF4093B

Commit message: Piezo wiring connections updated based on tests
Other:
- note added: "The ESD-48 uses a self-driven piezo speaker. The wiring connections are believed to be as follows: Green wire: Ground terminal (G) Red wire: Main terminal (M) White wire: Feedback terminal (F)"
- note removed: "The ESD-48 uses a self-driven piezo speaker. The wiring connections are likely as follows: Green wire: Main terminal (M) Red wire: Ground terminal (G) White wire: Feedback terminal (F)"
Changed lines of the file:
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@@
 		(company "trwgQ26xxx")
 	)
-	(text "The ESD-48 uses a self-driven piezo speaker.\n\nThe wiring connections are likely as follows:\n\nGreen wire: Main terminal (M)\nRed wire: Ground terminal (G)\nWhite wire: Feedback terminal (F)"
+	(text "The ESD-48 uses a self-driven piezo speaker.\n\nThe wiring connections are believed to be as follows:\n\nGreen wire: Ground terminal (G)\nRed wire: Main terminal (M)\nWhite wire: Feedback terminal (F)"
 		(exclude_from_sim no)
 		(at 228.854 107.442 0)
@@
 		)
 		(instances
-			(project ""
+			(project "ESD_48"
 				(path "/5035a11f-dc0a-45f5-8a5c-37f69c61abbb"
 					(reference "C2")
@@
 		)
 		(instances
-			(project ""
+			(project "ESD_48"
 				(path "/5035a11f-dc0a-45f5-8a5c-37f69c61abbb"
 					(reference "J1")
@@
 		)
 		(instances
-			(project ""
+			(project "ESD_48"
 				(path "/5035a11f-dc0a-45f5-8a5c-37f69c61abbb"
 					(reference "U1")
@@
 		)
 		(instances
-			(project ""
+			(project "ESD_48"
 				(path "/5035a11f-dc0a-45f5-8a5c-37f69c61abbb"
 					(reference "U1")
@@
 		)
 		(instances
-			(project ""
+			(project "ESD_48"
 				(path "/5035a11f-dc0a-45f5-8a5c-37f69c61abbb"
 					(reference "D1")
@@
 		)
 		(instances
-			(project ""
+			(project "ESD_48"
 				(path "/5035a11f-dc0a-45f5-8a5c-37f69c61abbb"
 					(reference "D2")
@@
 		)
 		(instances
-			(project ""
+			(project "ESD_48"
 				(path "/5035a11f-dc0a-45f5-8a5c-37f69c61abbb"
 					(reference "#PWR01")
@@
 		)
 		(instances
-			(project ""
+			(project "ESD_48"
 				(path "/5035a11f-dc0a-45f5-8a5c-37f69c61abbb"
 					(reference "U1")
@@
 		)
 		(instances
-			(project ""
+			(project "ESD_48"
 				(path "/5035a11f-dc0a-45f5-8a5c-37f69c61abbb"
 					(reference "U1")
@@
 		)
 		(instances
-			(project ""
+			(project "ESD_48"
 				(path "/5035a11f-dc0a-45f5-8a5c-37f69c61abbb"
 					(reference "C1")
@@
 		)
 		(instances
-			(project ""
+			(project "ESD_48"
 				(path "/5035a11f-dc0a-45f5-8a5c-37f69c61abbb"
 					(reference "R1")
@@
 		)
 		(instances
-			(project ""
+			(project "ESD_48"
 				(path "/5035a11f-dc0a-45f5-8a5c-37f69c61abbb"
 					(reference "U1")
